File: current shunt.brd (EAGLE design)
At the start: 40 x 50 mm, 46 parts, among them Q1 BC846,215, Q2 TIP29A, Q3 BC846,215, Q4 TIP29A

Commit message: update schematics to the version that was used for measurements in https://arxiv.org/abs/1808.03310
Parts:
- R9: value 20k -> 30k
Changed lines of the file:
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@@
 <?xml version="1.0" encoding="utf-8"?>
 <!DOCTYPE eagle SYSTEM "eagle.dtd">
-<eagle version="6.6.0">
+<eagle version="8.3.2">
 <drawing>
 <settings>
 <setting alwaysvectorfont="no"/>
+<setting keepoldvectorfont="yes"/>
 <setting verticaltext="up"/>
 </settings>
@@
 <layer number="54" name="bGND_GNDA" color="1" fill="9" visible="no" active="no"/>
 <layer number="56" name="wert" color="7" fill="1" visible="no" active="no"/>
-<layer number="90" name="Modules" color="5" fill="1" visible="no" active="yes"/>
+<layer number="90" name="Modules" color="5" fill="1" visible="no" active="no"/>
 <layer number="91" name="Nets" color="2" fill="1" visible="no" active="no"/>
 <layer number="92" name="Busses" color="1" fill="1" visible="no" active="no"/>
@@
 <pass name="Default">
 <param name="RoutingGrid" value="50mil"/>
+<param name="AutoGrid" value="1"/>
+<param name="Efforts" value="0"/>
+<param name="TopRouterVariant" value="1"/>
 <param name="tpViaShape" value="round"/>
 <param name="PrefDir.1" value="|"/>
@@
 <attribute name="VALUE" x="26.289" y="20.447" size="1.016" layer="27" rot="R270"/>
 </element>
-<element name="R9" library="custom-passive" package="0603" value="20k" x="29.718" y="17.78" smashed="yes" rot="R270">
+<element name="R9" library="custom-passive" package="0603" value="30k" x="29.718" y="17.78" smashed="yes" rot="R270">
 <attribute name="NAME" x="30.099" y="20.701" size="1.016" layer="25" rot="R90"/>
 <attribute name="VALUE" x="27.813" y="20.447" size="1.016" layer="27" rot="R270"/>
