File: current stabiliser.brd (EAGLE design)
At the start: 110 x 70 mm, 171 parts

Commit message: update schematics to the version that was used for measurements in https://arxiv.org/abs/1808.03310
Parts:
- removed R58, R59: 390R, custom-passive:0603
- R19: value 470R -> 270R
- R20: value 4k7 -> 9k1
- R21, R22: value 2k -> 3k6
- R24: value 1k -> 300R
- R56: value 0R -> 10R
- REF: value LTC6655LS8 -> LTC6655; device custom-ic:LS8 -> custom-ic:MSOP8
- moved R43 1.78 mm to (10.2, 54.6)
- moved R44 1.78 mm to (18.5, 54.6)
- moved REF 0.25 mm to (3.81, 49.0), turned to 0 degrees
Connections:
- net GND: no longer R58.2, R59.2
- net V_REF1_LP: no longer R58.1
- net V_REF2_LP: no longer R59.1
Routing:
- net V_REF2_LP: track 25.6 -> 22.6 mm
- net V_REF1_LP: track 25.1 -> 22.1 mm
- net V_REFBUF1: track 8.09 -> 9.87 mm
- net V_REF1A: track 8.35 -> 10.1 mm
- net GND: vias 231 -> 233
Other:
- board text added: "Current stabiliser main v4 BM Jul 2016"
- board text removed: "Current stabiliser main v4 - LS8 BM Jul 2016"
